File: KiCad/KVL/KVL.kicad_pcb (KiCad board)
At the start: 2 copper layers, 279.5 x 95 mm, 251 parts, among them J1 AudioJack2_Ground, J2 Conn_01x04, J3 AudioJack2_Ground, J4 Conn_01x11, SW1 SW_MEC_5G, SW10 SW_MEC_5G, SW11 SW_MEC_5G, SW12 SW_MEC_5G, SW13 SW_MEC_5G, SW14 SW_MEC_5G, SW15 SW_MEC_5G, SW16 SW_MEC_5G, SW17 SW_MEC_5G, SW18 SW_MEC_5G, SW19 SW_MEC_5G, SW2 SW_MEC_5G, SW20 SW_MEC_5G, SW21 SW_MEC_5G, SW22 SW_MEC_5G, SW23 SW_MEC_5G, SW24 SW_MEC_5G, SW25 SW_MEC_5G, SW26 SW_MEC_5G, SW27 SW_MEC_5G, SW28 SW_MEC_5G, SW29 SW_MEC_5G, SW3 SW_MEC_5G, SW30 SW_MEC_5G, SW31 SW_MEC_5G, SW32 SW_MEC_5G, SW33 SW_MEC_5G, SW34 SW_MEC_5G, SW35 SW_MEC_5G, SW36 SW_MEC_5G, SW37 SW_MEC_5G, SW38 SW_MEC_5G, SW39 SW_MEC_5G, SW4 SW_MEC_5G, SW40 SW_MEC_5G, SW41 SW_MEC_5G, SW42 SW_MEC_5G, SW43 SW_MEC_5G, SW44 SW_MEC_5G, SW45 SW_MEC_5G, SW46 SW_MEC_5G, SW47 SW_MEC_5G, SW48 SW_MEC_5G, SW49 SW_MEC_5G, SW5 SW_MEC_5G, SW50 SW_MEC_5G, SW51 SW_MEC_5G, SW52 SW_MEC_5G, SW53 SW_MEC_5G, SW54 SW_MEC_5G, SW55 SW_MEC_5G, SW56 SW_MEC_5G, SW57 SW_MEC_5G, SW58 SW_MEC_5G, SW59 SW_MEC_5G, SW6 SW_MEC_5G, SW60 SW_MEC_5G, SW61 SW_MEC_5G, SW62 SW_MEC_5G, SW63 SW_MEC_5G, SW64 SW_MEC_5G, SW65 SW_MEC_5G, SW7 SW_MEC_5G, SW8 SW_MEC_5G, SW9 SW_MEC_5G, U1 74HC164, U2 74HC165, U3 74HC165, U5 ADAU1761BCPZ, U6 MIC2005A-1YM5-TR

Commit message: 基板の寸法情報を追加
Other:
- board text added: "UNIT: mm PITCH: 2.54"
- board text added: "[J2] 1:PA9(I2C2_SCL) 2:PA8(I2C2_SDA) 3:RST for ADAU1761 4:GND"
- board text added: "[J4] 1:VCC 2:PA15(USART2_RX) 3:PA2 (USART2_TX) 4:PB15(SPI2_MOSI) 5:PB14(SPI2_MISO) 6:PF1 (SPI2_SCK) 7:PB13(ADC3_IN5) 8:PA4 (ADC2_IN17) 9:PA5 (ADC2_IN13) 10:PB2(ADC2_IN12) 11:GND"
Changed lines of the file:
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@@
     (effects (font (size 1.5 1.5) (thickness 0.2)) (justify left bottom mirror))
   )
+  (gr_text "[J2]\n1:PA9(I2C2_SCL)\n2:PA8(I2C2_SDA)\n3:RST for ADAU1761\n4:GND" (at 29.3 124.9) (layer "Cmts.User")
+    (effects (font (size 1 1) (thickness 0.15)) (justify left bottom))
+  )
+  (gr_text "UNIT: mm\nPITCH: 2.54" (at 29.3 94.2) (layer "Cmts.User")
+    (effects (font (size 1 1) (thickness 0.15)) (justify left bottom))
+  )
+  (gr_text "[J4]\n1:VCC\n2:PA15(USART2_RX)\n3:PA2 (USART2_TX)\n4:PB15(SPI2_MOSI)\n5:PB14(SPI2_MISO)\n6:PF1 (SPI2_SCK)\n7:PB13(ADC3_IN5)\n8:PA4 (ADC2_IN17)\n9:PA5 (ADC2_IN13)\n10:PB2(ADC2_IN12)\n11:GND" (at 29.3 114.8) (layer "Cmts.User")
+    (effects (font (size 1 1) (thickness 0.15)) (justify left bottom))
+  )
   (dimension (type aligned) (layer "Cmts.User")
-    (pts (xy 58.5 90.5) (xy 338 90.5))
-    (height -2.3)
-    (gr_text "279.5000 mm" (at 198.25 87.05) (layer "Cmts.User")
+    (pts (xy 318.5 90.6) (xy 223.5 90.6))
+    (height 2.2)
+    (gr_text "95.00" (at 271 87.25) (layer "Cmts.User")
       (effects (font (size 1 1) (thickness 0.15)))
     )
-    (format (prefix "") (suffix "") (units 3) (units_format 1) (precision 4))
+    (format (prefix "") (suffix "") (units 3) (units_format 0) (precision 2))
     (style (thickness 0.15) (arrow_length 1.27) (text_position_mode 0) (extension_height 0.58642) (extension_offset 0.5) keep_text_aligned)
   )
   (dimension (type aligned) (layer "Cmts.User")
-    (pts (xy 58.5 185.5) (xy 58.5 90.5))
-    (height -2.7)
-    (gr_text "95.0000 mm" (at 54.65 138 90) (layer "Cmts.User")
+    (pts (xy 109.5 90.6) (xy 61 90.6))
+    (height 2.2)
+    (gr_text "48.50" (at 85.25 87.25) (layer "Cmts.User")
       (effects (font (size 1 1) (thickness 0.15)))
     )
-    (format (prefix "") (suffix "") (units 3) (units_format 1) (precision 4))
+    (format (prefix "") (suffix "") (units 3) (units_format 0) (precision 2))
     (style (thickness 0.15) (arrow_length 1.27) (text_position_mode 0) (extension_height 0.58642) (extension_offset 0.5) keep_text_aligned)
   )
+  (dimension (type aligned) (layer "Cmts.User")
+    (pts (xy 109.5 90.6) (xy 204.5 90.6))
+    (height -2.2)
+    (gr_text "95.00" (at 157 87.25) (layer "Cmts.User")
+      (effects (font (size 1 1) (thickness 0.15)))
+    )
+    (format (prefix "") (suffix "") (units 3) (units_format 0) (precision 2))
+    (style (thickness 0.15) (arrow_length 1.27) (text_position_mode 0) (extension_height 0.58642) (extension_offset 0.5) keep_text_aligned)
+  )
+  (dimension (type aligned) (layer "Cmts.User")
+    (pts (xy 223.5 90.6) (xy 204.5 90.6))
+    (height 2.2)
+    (gr_text "19.00" (at 214 87.25) (layer "Cmts.User")
+      (effects (font (size 1 1) (thickness 0.15)))
+    )
+    (format (prefix "") (suffix "") (units 3) (units_format 0) (precision 2))
+    (style (thickness 0.15) (arrow_length 1.27) (text_position_mode 0) (extension_height 0.58642) (extension_offset 0.5) keep_text_aligned)
+  )
+  (dimension (type aligned) (layer "Cmts.User")
+    (pts (xy 61 165) (xy 61 183))
+    (height 4.7)
+    (gr_text "18.00" (at 55.15 174 90) (layer "Cmts.User")
+      (effects (font (size 1 1) (thickness 0.15)))
+    )
+    (format (prefix "") (suffix "") (units 3) (units_format 0) (precision 2))
+    (style (thickness 0.15) (arrow_length 1.27) (text_position_mode 0) (extension_height 0.58642) (extension_offset 0.5) keep_text_aligned)
+  )
+  (dimension (type aligned) (layer "Cmts.User")
+    (pts (xy 318.5 90.6) (xy 338 90.6))
+    (height -2.2)
+    (gr_text "19.50" (at 328.25 87.25) (layer "Cmts.User")
+      (effects (font (size 1 1) (thickness 0.15)))
+    )
+    (format (prefix "") (suffix "") (units 3) (units_format 0) (precision 2))
+    (style (thickness 0.15) (arrow_length 1.27) (text_position_mode 0) (extension_height 0.58642) (extension_offset 0.5) keep_text_aligned)
+  )
+  (dimension (type aligned) (layer "Cmts.User")
+    (pts (xy 58.5 185.5) (xy 58.5 183))
+    (height -2.2)
+    (gr_text "2.50" (at 55.15 184.25 90) (layer "Cmts.User")
+      (effects (font (size 1 1) (thickness 0.15)))
+    )
+    (format (prefix "") (suffix "") (units 3) (units_format 0) (precision 2))
+    (style (thickness 0.15) (arrow_length 1.27) (text_position_mode 0) (extension_height 0.58642) (extension_offset 0.5) keep_text_aligned)
+  )
+  (dimension (type aligned) (layer "Cmts.User")
+    (pts (xy 58.5 90.5) (xy 61 90.5))
+    (height -2.1)
+    (gr_text "2.50" (at 59.75 87.25) (layer "Cmts.User")
+      (effects (font (size 1 1) (thickness 0.15)))
+    )
+    (format (prefix "") (suffix "") (units 3) (units_format 0) (precision 2))
+    (style (thickness 0.15) (arrow_length 1.27) (text_position_mode 0) (extension_height 0.58642) (extension_offset 0.5) keep_text_aligned)
+  )
+  (dimension (type aligned) (layer "Cmts.User")
+    (pts (xy 58.5 87.8) (xy 338 87.8))
+    (height -3.1)
+    (gr_text "279.50" (at 198.25 83.55) (layer "Cmts.User")
+      (effects (font (size 1 1) (thickness 0.15)))
+    )
+    (format (prefix "") (suffix "") (units 3) (units_format 0) (precision 2))
+    (style (thickness 0.15) (arrow_length 1.27) (text_position_mode 0) (extension_height 0.58642) (extension_offset 0.5) keep_text_aligned)
+  )
+  (dimension (type orthogonal) (layer "Cmts.User")
+    (pts (xy 61 165) (xy 204.475 147.475))
+    (height -4.7)
+    (orientation 1)
+    (gr_text "17.5250" (at 55.15 156.2375 90) (layer "Cmts.User")
+      (effects (font (size 1 1) (thickness 0.15)))
+    )
+    (format (prefix "") (suffix "") (units 3) (units_format 0) (precision 4))
+    (style (thickness 0.15) (arrow_length 1.27) (text_position_mode 0) (extension_height 0.58642) (extension_offset 0.5) keep_text_aligned)
+  )
+  (dimension (type orthogonal) (layer "Cmts.User")
+    (pts (xy 58.5 185.5) (xy 58.5 90.5))
+    (height -6.6)
+    (orientation 1)
+    (gr_text "95.00" (at 50.75 138 90) (layer "Cmts.User")
+      (effects (font (size 1 1) (thickness 0.15)))
+    )
+    (format (prefix "") (suffix "") (units 3) (units_format 0) (precision 2))
+    (style (thickness 0.15) (arrow_length 1.27) (text_position_mode 0) (extension_height 0.58642) (extension_offset 0.5) keep_text_aligned)
+  )
+  (dimension (type orthogonal) (layer "Cmts.User")
+    (pts (xy 109.525 109.475) (xy 61 93))
+    (height -53.225)
+    (orientation 1)
+    (gr_text "16.4750" (at 55.15 101.2375 90) (layer "Cmts.User")
+      (effects (font (size 1 1) (thickness 0.15)))
+    )
+    (format (prefix "") (suffix "") (units 3) (units_format 0) (precision 4))
+    (style (thickness 0.15) (arrow_length 1.27) (text_position_mode 0) (extension_height 0.58642) (extension_offset 0.5) keep_text_aligned)
+  )
+  (dimension (type orthogonal) (layer "Cmts.User")
+    (pts (xy 61 93) (xy 58.5 90.5))
+    (height -4.7)
+    (orientation 1)
+    (gr_text "2.50" (at 55.15 91.75 90) (layer "Cmts.User")
+      (effects (font (size 1 1) (thickness 0.15)))
+    )
+    (format (prefix "") (suffix "") (units 3) (units_format 0) (precision 2))
+    (style (thickness 0.15) (arrow_length 1.27) (text_position_mode 0) (extension_height 0.58642) (extension_offset 0.5) keep_text_aligned)
+  )
+  (dimension (type orthogonal) (layer "Cmts.User")
+    (pts (xy 223.525 128.475) (xy 109.475 109.475))
+    (height -167.225)
+    (orientation 1)
+    (gr_text "19.00" (at 55.15 118.975 90) (layer "Cmts.User")
+      (effects (font (size 1 1) (thickness 0.15)))
+    )
+    (format (prefix "") (suffix "") (units 3) (units_format 0) (precision 2))
+    (style (thickness 0.15) (arrow_length 1.27) (text_position_mode 0) (extension_height 0.58642) (extension_offset 0.5) keep_text_aligned)
+  )
+  (dimension (type orthogonal) (layer "Cmts.User")
+    (pts (xy 204.475 147.525) (xy 223.475 128.475))
+    (height -148.175)
+    (orientation 1)
+    (gr_text "19.05" (at 55.15 138 90) (layer "Cmts.User")
+      (effects (font (size 1 1) (thickness 0.15)))
+    )
+    (format (prefix "") (suffix "") (units 3) (units_format 0) (precision 2))
+    (style (thickness 0.15) (arrow_length 1.27) (text_position_mode 0) (extension_height 0.58642) (extension_offset 0.5) keep_text_aligned)
+  )

Commit message: キースイッチをソケット化
Parts:
- RV1, RV2: footprint My_Parts:PTV09A4015UB103 -> My_Parts:RK09K1130A5R
- SW1, SW10, SW11, SW12, SW13, SW14, SW15, SW16, SW17, SW18, SW19, SW2, SW20, SW21, SW22, SW23, SW24, SW25, SW26, SW27, SW28, SW29, SW3, SW30, SW31, SW32, SW33, SW34, SW35, SW36, SW37, SW38, SW39, SW4, SW40, SW41, SW42, SW43, SW44, SW45, SW46, SW47, SW48, SW49, SW5, SW50, SW51, SW52, SW53, SW54, SW55, SW56, SW57, SW58, SW59, SW6, SW60, SW61, SW62, SW63, SW64, SW65, SW7, SW8, SW9: footprint My_Parts:Gateron Low Profile Switch 2.0 -> My_Parts:Gateron_KS-27; moved to B.Cu
- moved D16 10.1 mm to (133.6, 117.0), turned to -90 degrees
- moved D17 10.1 mm to (152.6, 117.0), turned to -90 degrees
- moved D18 10.1 mm to (171.6, 117.0), turned to -90 degrees
- moved D19 10.1 mm to (190.6, 117.0), turned to -90 degrees
- moved D20 10.1 mm to (209.6, 117.0), turned to -90 degrees
- moved D21 10.1 mm to (228.6, 117.0), turned to -90 degrees
- moved D22 10.1 mm to (247.6, 117.0), turned to -90 degrees
- moved D14 10.1 mm to (95.6, 117.0), turned to -90 degrees
- moved D15 10.1 mm to (114.6, 117.0), turned to -90 degrees
- moved D23 10.1 mm to (266.6, 117.0), turned to -90 degrees
- moved D24 10.1 mm to (285.6, 117.0), turned to -90 degrees
- moved D25 10.1 mm to (304.6, 117.0), turned to -90 degrees
- moved D26 10.1 mm to (323.6, 117.0), turned to -90 degrees
- moved D55 9.84 mm to (133.7, 174.2), turned to -90 degrees
- moved D56 9.84 mm to (152.7, 174.2), turned to -90 degrees
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- renumbered REF** to MH1, REF** to MH2, REF** to MH3, REF** to MH4, REF** to MH5, REF** to MH6, REF** to MH7, REF** to MH8, REF** to MH9
Routing:
- net Q4: track 100.6 -> 165.5 mm, vias 1 -> 5
- net VCC: track 314.8 -> 379.2 mm, vias 5 -> 4
- net Q0_2: track 139.2 -> 194.7 mm, vias 2 -> 5
- net Q3_2: track 113.9 -> 166.9 mm, vias 1 -> 7
- net Q7: track 157.3 -> 206.4 mm, vias 1 -> 6
- net Q6: track 143.0 -> 188.7 mm, vias 3 -> 8
- net Q1: track 154.3 -> 198.6 mm, vias 1 -> 6
- net Q2_2: track 100.3 -> 144.2 mm, vias 1 -> 6
- net Q5: track 126.0 -> 169.3 mm, vias 4 -> 8
- net Q0: track 183.4 -> 222.5 mm, vias 4 -> 10
- net Q4_2: track 154.5 -> 191.8 mm, vias 0 -> 5
- net Q1_2: track 114.4 -> 145.5 mm, vias 1 -> 6
- net Q3: track 110.5 -> 136.9 mm, vias 1 -> 6
- net QE: track 298.8 -> 274.8 mm, vias 4 -> 2
- net QD: track 282.7 -> 269.7 mm, vias 4 -> 2
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Other:
- board text added: "RST"
- board text added: "SCL"
- board text added: "SDA"
