File: KiCad/KVL/KVL.kicad_sch (KiCad schematic)
At the start: 195 parts, among them SW1 SW_MEC_5G, SW10 SW_MEC_5G, SW11 SW_MEC_5G, SW12 SW_MEC_5G, SW13 SW_MEC_5G, SW14 SW_MEC_5G, SW15 SW_MEC_5G, SW16 SW_MEC_5G, SW17 SW_MEC_5G, SW18 SW_MEC_5G, SW19 SW_MEC_5G, SW2 SW_MEC_5G, SW20 SW_MEC_5G, SW21 SW_MEC_5G, SW22 SW_MEC_5G, SW23 SW_MEC_5G, SW24 SW_MEC_5G, SW25 SW_MEC_5G, SW26 SW_MEC_5G, SW27 SW_MEC_5G, SW28 SW_MEC_5G, SW29 SW_MEC_5G, SW3 SW_MEC_5G, SW30 SW_MEC_5G, SW31 SW_MEC_5G, SW32 SW_MEC_5G, SW33 SW_MEC_5G, SW34 SW_MEC_5G, SW35 SW_MEC_5G, SW36 SW_MEC_5G, SW37 SW_MEC_5G, SW38 SW_MEC_5G, SW39 SW_MEC_5G, SW4 SW_MEC_5G, SW40 SW_MEC_5G, SW41 SW_MEC_5G, SW42 SW_MEC_5G, SW43 SW_MEC_5G, SW44 SW_MEC_5G, SW45 SW_MEC_5G, SW46 SW_MEC_5G, SW47 SW_MEC_5G, SW48 SW_MEC_5G, SW49 SW_MEC_5G, SW5 SW_MEC_5G, SW50 SW_MEC_5G, SW51 SW_MEC_5G, SW52 SW_MEC_5G, SW53 SW_MEC_5G, SW54 SW_MEC_5G, SW55 SW_MEC_5G, SW56 SW_MEC_5G, SW57 SW_MEC_5G, SW58 SW_MEC_5G, SW59 SW_MEC_5G, SW6 SW_MEC_5G, SW60 SW_MEC_5G, SW61 SW_MEC_5G, SW62 SW_MEC_5G, SW63 SW_MEC_5G, SW64 SW_MEC_5G, SW65 SW_MEC_5G, SW7 SW_MEC_5G, SW8 SW_MEC_5G, SW9 SW_MEC_5G

Commit message: キースイッチをソケット化
Parts:
- SW1, SW10, SW11, SW12, SW13, SW14, SW15, SW16, SW17, SW18, SW19, SW2, SW20, SW21, SW22, SW23, SW24, SW25, SW26, SW27, SW28, SW29, SW3, SW30, SW31, SW32, SW33, SW34, SW35, SW36, SW37, SW38, SW39, SW4, SW40, SW41, SW42, SW43, SW44, SW45, SW46, SW47, SW48, SW49, SW5, SW50, SW51, SW52, SW53, SW54, SW55, SW56, SW57, SW58, SW59, SW6, SW60, SW61, SW62, SW63, SW64, SW65, SW7, SW8, SW9: footprint My_Parts:Gateron Low Profile Switch 2.0 -> My_Parts:Gateron_KS-27
